File: sch/iqboard.sch (KiCad schematic (older format))
At the start: 33 parts, among them T1 TRANSFO4, U3 TLE2426CP, U4 SN74CBTLV3253D, U5 LT6231CS8, U6 LT6231CS8, U7 LT6231CS8

Commit message: add FIN1002 buffer for LVDS variant of Si570
Parts:
- removed R3, R7: 10k, symbol R
- renumbered R12 to R10, R13 to R11, R14 to R12, R15 to R13, R16 to R14, R4 to R3, R5 to R4, R6 to R5, R8 to R6, R9 to R7, R10 to R8, R11 to R9, U3 to U1, U4 to U2, U5 to U3, U6 to U4, U7 to U5
Changed lines of the file:
@@
-EESchema Schematic File Version 2  date so 30 črv 00:27:21 2012
+EESchema Schematic File Version 2  date so 30 črv 11:50:59 2012
 LIBS:power
 LIBS:device
@@
 LIBS:ms-audio
 LIBS:ms-conn
+LIBS:ms-ti
+LIBS:hf-sampling-trx-cache
 EELAYER 25  0
 EELAYER END
 $Descr A4 11693 8268
 encoding utf-8
-Sheet 3 4
+Sheet 3 5
 Title "noname.sch"
-Date "29 jun 2012"
+Date "30 jun 2012"
 Rev ""
 Comp ""
@@
 bias
 $Comp
-L R R14
+L R R12
 U 1 1 4FEDB599
 P 10000 2900
-F 0 "R14" V 10080 2900 50  0000 C CNN
+F 0 "R12" V 10080 2900 50  0000 C CNN
 F 1 "R" V 10000 2900 50  0000 C CNN
 	1    10000 2900
@@
 $EndComp
 $Comp
-L R R10
+L R R8
 U 1 1 4FEDB597
 P 8650 2900
-F 0 "R10" V 8730 2900 50  0000 C CNN
+F 0 "R8" V 8730 2900 50  0000 C CNN
 F 1 "R" V 8650 2900 50  0000 C CNN
 	1    8650 2900
@@
 $EndComp
 $Comp
-L R R13
+L R R11
 U 1 1 4FEDB593
 P 10000 1400
-F 0 "R13" V 10080 1400 50  0000 C CNN
+F 0 "R11" V 10080 1400 50  0000 C CNN
 F 1 "R" V 10000 1400 50  0000 C CNN
 	1    10000 1400
@@
 $EndComp
 $Comp
-L R R9
+L R R7
 U 1 1 4FEDB58F
 P 8650 1400
-F 0 "R9" V 8730 1400 50  0000 C CNN
+F 0 "R7" V 8730 1400 50  0000 C CNN
 F 1 "R" V 8650 1400 50  0000 C CNN
 	1    8650 1400
@@
 $EndComp
 $Comp
-L R R5
+L R R4
 U 1 1 4FEDB48A
 P 8300 2650
-F 0 "R5" V 8380 2650 50  0000 C CNN
+F 0 "R4" V 8380 2650 50  0000 C CNN
 F 1 "10k" V 8300 2650 50  0000 C CNN
 	1    8300 2650
@@
 $EndComp
 $Comp
-L R R4
+L R R3
 U 1 1 4FEDB482
 P 8300 1650
-F 0 "R4" V 8380 1650 50  0000 C CNN
+F 0 "R3" V 8380 1650 50  0000 C CNN
 F 1 "10k" V 8300 1650 50  0000 C CNN
 	1    8300 1650
@@
 $EndComp
 $Comp
-L LT6231CS8 U7
+L LT6231CS8 U5
 U 1 1 4FEDB3CD
 P 9600 2100
-F 0 "U7" H 9150 2400 60  0000 C CNN
+F 0 "U5" H 9150 2400 60  0000 C CNN
 F 1 "LT6231CS8" H 9300 2500 60  0000 C CNN
 	1    9600 2100
@@
 $EndComp
 $Comp
-L TLE2426CP U3
+L TLE2426CP U1
 U 1 1 4FEC43DB
 P 2050 3900
-F 0 "U3" H 2300 4200 60  0000 C CNN
+F 0 "U1" H 2300 4200 60  0000 C CNN
 F 1 "TLE2426CP" H 2050 3900 60  0000 C CNN
 	1    2050 3900
@@
 $EndComp
 $Comp
-L LT6231CS8 U5
+L LT6231CS8 U3
 U 1 1 4FEC435B
 P 7550 1400
-F 0 "U5" H 7100 1700 60  0000 C CNN
+F 0 "U3" H 7100 1700 60  0000 C CNN
 F 1 "LT6231CS8" H 7250 1800 60  0000 C CNN
 	1    7550 1400
@@
 	1    1600 1950
 	0    -1   -1   0
-$EndComp
-$Comp
-L R R3
-U 1 1 4FEC4356
-P 8300 1650
-F 0 "R3" V 8380 1650 50  0000 C CNN
-F 1 "10k" V 8300 1650 50  0000 C CNN
-	1    8300 1650
-	1    0    0    -1
 $EndComp
 $Comp
@@
 $EndComp
 $Comp
-L SN74CBTLV3253D U4
+L SN74CBTLV3253D U2
 U 1 1 4FEC434C
 P 3950 1800
-F 0 "U4" H 4250 2600 60  0000 C CNN
+F 0 "U2" H 4250 2600 60  0000 C CNN
 F 1 "SN74CBTLV3253D" H 3950 1800 60  0000 C CNN
 	1    3950 1800
@@
 GND
 $Comp
-L LT6231CS8 U5
+L LT6231CS8 U3
 U 2 1 4FEDB3BC
 P 7550 2900
-F 0 "U5" H 7100 3200 60  0000 C CNN
+F 0 "U3" H 7100 3200 60  0000 C CNN
 F 1 "LT6231CS8" H 7250 3300 60  0000 C CNN
 	2    7550 2900
@@
 bias
 $Comp
-L R R16
+L R R14
 U 1 1 4FEE032D
 P 10000 6100
-F 0 "R16" V 10080 6100 50  0000 C CNN
+F 0 "R14" V 10080 6100 50  0000 C CNN
 F 1 "R" V 10000 6100 50  0000 C CNN
 	1    10000 6100
@@
 $EndComp
 $Comp
-L R R12
+L R R10
 U 1 1 4FEE0333
 P 8650 6100
-F 0 "R12" V 8730 6100 50  0000 C CNN
+F 0 "R10" V 8730 6100 50  0000 C CNN
 F 1 "R" V 8650 6100 50  0000 C CNN
 	1    8650 6100
@@
 $EndComp
 $Comp
-L R R15
+L R R13
 U 1 1 4FEE0339
 P 10000 4600
-F 0 "R15" V 10080 4600 50  0000 C CNN
+F 0 "R13" V 10080 4600 50  0000 C CNN
 F 1 "R" V 10000 4600 50  0000 C CNN
 	1    10000 4600
@@
 $EndComp
 $Comp
-L R R11
+L R R9
 U 1 1 4FEE033F
 P 8650 4600
-F 0 "R11" V 8730 4600 50  0000 C CNN
+F 0 "R9" V 8730 4600 50  0000 C CNN
 F 1 "R" V 8650 4600 50  0000 C CNN
 	1    8650 4600
@@
 $EndComp
 $Comp
-L R R8
+L R R6
 U 1 1 4FEE034B
 P 8300 5850
-F 0 "R8" V 8380 5850 50  0000 C CNN
+F 0 "R6" V 8380 5850 50  0000 C CNN
 F 1 "10k" V 8300 5850 50  0000 C CNN
 	1    8300 5850
@@
 $EndComp
 $Comp
-L R R6
+L R R5
 U 1 1 4FEE0351
 P 8300 4850
-F 0 "R6" V 8380 4850 50  0000 C CNN
+F 0 "R5" V 8380 4850 50  0000 C CNN
 F 1 "10k" V 8300 4850 50  0000 C CNN
 	1    8300 4850
@@
 $EndComp
 $Comp
-L LT6231CS8 U7
+L LT6231CS8 U5
 U 2 1 4FEE0357
 P 9600 5300
-F 0 "U7" H 9150 5600 60  0000 C CNN
+F 0 "U5" H 9150 5600 60  0000 C CNN
 F 1 "LT6231CS8" H 9300 5700 60  0000 C CNN
 	2    9600 5300
@@
 $EndComp
 $Comp
-L LT6231CS8 U6
+L LT6231CS8 U4
 U 1 1 4FEE035D
 P 7550 4600
-F 0 "U6" H 7100 4900 60  0000 C CNN
+F 0 "U4" H 7100 4900 60  0000 C CNN
 F 1 "LT6231CS8" H 7250 5000 60  0000 C CNN
 	1    7550 4600
-	1    0    0    -1
-$EndComp
-$Comp
-L R R7
-U 1 1 4FEE0363
-P 8300 4850
-F 0 "R7" V 8380 4850 50  0000 C CNN
-F 1 "10k" V 8300 4850 50  0000 C CNN
-	1    8300 4850
 	1    0    0    -1
 $EndComp
@@
 $EndComp
 $Comp
-L LT6231CS8 U6
+L LT6231CS8 U4
 U 2 1 4FEE0378
 P 7550 6100
-F 0 "U6" H 7100 6400 60  0000 C CNN
+F 0 "U4" H 7100 6400 60  0000 C CNN
 F 1 "LT6231CS8" H 7250 6500 60  0000 C CNN
 	2    7550 6100
