File: sch/cpu.sch (KiCad schematic (older format))
At the start: 36 parts

Commit message: Add models and updated schematics
Parts:
- removed C? (x2): 100n, symbol C
- removed C? (x2): 10n, symbol C
- removed C? (x4): C, symbol C
- removed CONN?: 3.5\"_STEREO_JACK, symbol 3.5"_STEREO_JACK
- removed R?: 100, symbol R
- removed R? (x4): R, symbol R
- removed U?: LP2992AIM5-5.0V, SOT23-5, symbol LP2992AIM5-3.3V
- removed U?: LP2992AIM5-3.3V, SOT23-5, symbol LP2992AIM5-3.3V
- removed U?: TPA6111A2D, symbol TPA6111A2D
- removed U?: DS1807, symbol DS1807
- removed U?: XC9572XL-PC44, symbol XC9572XL-PC44
- removed U?: SI570, symbol SI570
- removed U?: FIN1002, symbol FIN1002
- removed U?: MSP430G2553-20, symbol MSP430G2XX3-20
- removed U?: SN74CBTLV3253D, symbol SN74CBTLV3253D
- added IC?: ATXMEGA256A3B-A, TQFP64, symbol ATXMEGA256A3B-A
Connections:
- net labels added: CLK, DATA, KEYA, KEYB, PROG_CLK, PROG_DATA, RX, TX
- net labels removed: +5V, SCL, SDA, VCC
- wire segments 82 -> 75
- no-connect marks 1 -> 0
Other:
- note added: "ADC channels (less tham 1Msps, Vref less than 2.4V, differential mode)\nreceiver I\nreceiver Q\nFWD from SWR bridge\nREFL from SWR bridge\nPHASE from SWR phase detector\n\nAnalog Comparator\nzero detection for frequency counting (from oscillator)\n\nDAC (Vref less than 2.4V, se errata)\n- stereo output"
- note removed: "CMOS version of Si570 does not need the\n100R resistor and FIN1002 receiver\n- leave the resistor out\n- connect pins 3 and 5 of FIN1002's pads together"
