File: sch/lcd_rotary.sch (KiCad schematic (older format))
At the start: 0 parts

Commit message: Add models and updated schematics
Parts:
- added D1: BX56-12, symbol BX56-12
- added D2: DC-10, symbol DC-10
Connections:
- wire segments 0 -> 19
Changed lines of the file:
@@
-EESchema Schematic File Version 2  date 11/12/2012 10:11:24 PM
+EESchema Schematic File Version 2  date 3/16/2013 7:50:18 PM
 LIBS:power
 LIBS:device
@@
 LIBS:contrib
 LIBS:valves
-LIBS:cpu_power-cache
-EELAYER 25  0
+LIBS:ms-parts
+LIBS:ms-conn
+LIBS:ms-opto
+LIBS:lcd_rotary-cache
+EELAYER 27 0
 EELAYER END
-$Descr A4 11700 8267
+$Descr A4 11693 8268
 encoding utf-8
 Sheet 1 1
 Title "noname.sch"
-Date "12 nov 2012"
+Date "16 mar 2013"
 Rev ""
 Comp ""
@@
 Comment4 ""
 $EndDescr
+$Comp
+L DC-10 D2
+U 1 1 5141264E
+P 3600 6950
+F 0 "D2" H 3750 8400 60  0000 C CNN
+F 1 "DC-10" H 3400 8400 60  0000 C CNN
+F 2 "" H 3600 7600 60  0000 C CNN
+F 3 "" H 3600 7600 60  0000 C CNN
+	1    3600 6950
+	0    -1   -1   0
+$EndComp
+$Comp
+L BX56-12 D1
+U 1 1 5141265D
+P 1250 1200
+F 0 "D1" H 1800 1900 60  0000 C CNN
+F 1 "BX56-12" H 1100 1900 60  0000 C CNN
+F 2 "" H 1250 1200 60  0000 C CNN
+F 3 "" H 1250 1200 60  0000 C CNN
+	1    1250 1200
+	-1   0    0    -1
+$EndComp
+$Comp
+L BX56-12 D1
+U 2 1 5141266A
+P 1250 2700
+F 0 "D1" H 1800 3400 60  0000 C CNN
+F 1 "BX56-12" H 1100 3400 60  0000 C CNN
+F 2 "" H 1250 2700 60  0000 C CNN
+F 3 "" H 1250 2700 60  0000 C CNN
+	2    1250 2700
+	-1   0    0    -1
+$EndComp
+$Comp
+L BX56-12 D1
+U 3 1 51412670
+P 1250 5700
+F 0 "D1" H 1800 6400 60  0000 C CNN
+F 1 "BX56-12" H 1100 6400 60  0000 C CNN
+F 2 "" H 1250 5700 60  0000 C CNN
+F 3 "" H 1250 5700 60  0000 C CNN
+	3    1250 5700
+	-1   0    0    -1
+$EndComp
+Wire Wire Line
+	1950 1650 2300 1650
+Wire Wire Line
+	2300 3150 1950 3150
+Connection ~ 4450 7350
+Connection ~ 4200 7350
+Connection ~ 3950 7350
+Connection ~ 3700 7350
+Connection ~ 3450 7350
+Connection ~ 3200 7350
+Connection ~ 2950 7350
+Connection ~ 2700 7350
+Connection ~ 2450 7350
+Wire Wire Line
+	1950 800  2600 800
+Wire Wire Line
+	1950 900  2600 900
+Wire Wire Line
+	1950 1000 2600 1000
+Wire Wire Line
+	1950 1100 2600 1100
+Wire Wire Line
+	1950 1200 2600 1200
+Wire Wire Line
+	1950 1300 2600 1300
+Wire Wire Line
+	1950 1400 2600 1400
+Wire Wire Line
+	1950 1500 2600 1500
+Wire Wire Line
+	1950 2300 2600 2300
+Wire Wire Line
+	1950 2400 2600 2400
+Wire Wire Line
+	1950 2500 2600 2500
+Wire Wire Line
+	1950 2600 2600 2600
+Wire Wire Line
+	1950 2700 2600 2700
+Wire Wire Line
+	1950 2800 2600 2800
+Wire Wire Line
+	1950 2900 2600 2900
+Wire Wire Line
+	1950 3000 2600 3000
+Wire Wire Line
+	4700 7350 2450 7350
 $EndSCHEMATC
