File: sch/transmitter_bpf.sch (KiCad schematic (older format))
At the start: 42 parts

Commit message: Add models and updated schematics
Parts:
- added C? (x7): C, symbol C
- added K?: CONN_3, symbol CONN_3
- added L? (x3): INDUCTOR_WITH_CORE, symbol INDUCTOR_WITH_CORE
- added P? (x2): BNC, symbol BNC
- added P?: CONN_4, symbol CONN_4
- added P?: CONN_2, symbol CONN_2
- added Q? (x2): MOSFET_N, symbol MOSFET_N
- added R?: R, symbol R
- added U?: SN65LVDS2DBV, symbol SN65LVDS2DBV
Connections:
- net labels added: RX_OPEN_TX_GND, TX_OPEN_RX_GND, VCC
- wire segments 91 -> 119
Other:
- note added: "Antenna"
- note added: "Power connector"
- note added: "TXEN, PTT, RXEN\nsignals"
- note added: "differential I/Q\nclock from CPU board"
- note added: "to RX board"
- note removed: "TODO\ndoplnit BPF"
- moved on the sheet: C?, L?, Q?, R?
