File: sch/rx.sch (KiCad schematic (older format))
At the start: 43 parts, among them P1 FromBPF

Commit message: Add models and updated schematics
Parts:
- removed C12: CP1, symbol CP1
- removed C?: 100n, symbol C
- removed C?: 10n, symbol C
- removed CONN1: 3.5\"_STEREO_JACK, symbol 3.5"_STEREO_JACK
- removed U?: LP2992AIM5-3.3V, SOT23-5, symbol LP2992AIM5-3.3V
- added C?: C, symbol C
- added C?: 100n, symbol C
- added C?: 10n, symbol C
- added K? (x2): CONN_3, symbol CONN_3
- added P?: CONN_4, symbol CONN_4
- added P?: CONN_2, symbol CONN_2
- added R?: R, symbol R
- added R? (x4): 833, symbol R
- added U? (x2): SN65LVDS2DBV, symbol SN65LVDS2DBV
- added U?: LP2992AIM5-3.3V, SOT23-5, symbol LP2992AIM5-3.3V
- U?: value SN74CBTLV3253D -> SN74CBT3253D
Connections:
- net labels removed: /EN, 12V, SCL, SDA, clkA, clkB
- wire segments 122 -> 143
Other:
- note added: "2x\nHigh precision differential amplifiers\nsee A.13.3 (page A-17)\nin Opamps for everyone\n\n- high input impedance\n- high CMRR"
- note added: "I/Q audio\noutput"
- note added: "Input offset current prevention\n(omit or recalculate for ultra low noise?)"
- note added: "Power connector"
- note added: "Quadrature sampling detector\n(aka Tayloe detector)"
- note added: "RF input"
- note added: "RF input impedance\n(might not be needed)"
- note added: "TXEN, PTT and RXEN\ncontrol lines"
- note added: "differential I/Q clock\nfrom oscillator board"
- note added: "gain\nresistor"
- note added: "input from counter\nuses 1, 2, 4, 3 sequence"
- note removed: "CPLD counter has 1, 2, 3, 4 sequence"
- note removed: "Konektor bude obsahovat:\n\nSDA\nSCL\n+5V\n+3.3V\nTX\nTXEN\nGND"
- moved on the sheet: C?, P1, R?, T?, U?

Commit message: Prototype RX pcb
Parts:
- removed R?: R, symbol R
- C10, C11, C12, C9: renamed from C?; value 0.22u -> 820n
- R1, R2: renamed from R?; value R -> 5k1
- gave numbers to parts that had none: 42
Connections:
- no-connect marks 0 -> 1
Other:
- note added: "Cs 820n == BW 3.8kHz"
- note added: "Detector bandwidth\nBW (Hz) = 1 / (pi * N * Rant * Cs)\nN = number of phases / number of simultaneously active Cs\n(4 for single balanced, 2 for doubly balanced QSD)"
- note removed: "RF input impedance\n(might not be needed)"

Commit message: Add capacitors to RX board schematics
Parts:
- added C? (x2): C, ~, symbol C
Changed lines of the file:
@@
-EESchema Schematic File Version 2  date 3/24/2013 11:54:54 AM
+EESchema Schematic File Version 2  date ne 24 bře 22:39:58 2013
 LIBS:power
 LIBS:device
@@
 Title "QSD transceiver - RX board"
 Date "24 mar 2013"
-Rev "D"
+Rev "E"
 Comp ""
 Comment1 ""
@@
 Connection ~ 3650 1950
 Connection ~ 3650 950
+$Comp
+L C C?
+U 1 1 514F73A0
+P 4400 3650
+F 0 "C?" H 4400 3750 40  0000 L CNN
+F 1 "C" H 4406 3565 40  0000 L CNN
+F 2 "~" H 4438 3500 30  0000 C CNN
+F 3 "~" H 4400 3650 60  0000 C CNN
+	1    4400 3650
+	1    0    0    -1
+$EndComp
+$Comp
+L C C?
+U 1 1 514F73AD
+P 4400 4600
+F 0 "C?" H 4400 4700 40  0000 L CNN
+F 1 "C" H 4406 4515 40  0000 L CNN
+F 2 "~" H 4438 4450 30  0000 C CNN
+F 3 "~" H 4400 4600 60  0000 C CNN
+	1    4400 4600
+	1    0    0    -1
+$EndComp
+$Comp
+L +3.3V #PWR?
+U 1 1 514F73B5
+P 4400 4400
+F 0 "#PWR?" H 4400 4360 30  0001 C CNN
+F 1 "+3.3V" H 4400 4510 30  0000 C CNN
+F 2 "" H 4400 4400 60  0000 C CNN
+F 3 "" H 4400 4400 60  0000 C CNN
+	1    4400 4400
+	1    0    0    -1
+$EndComp
+$Comp
+L +3.3V #PWR?
+U 1 1 514F73C4
+P 4400 3450
+F 0 "#PWR?" H 4400 3410 30  0001 C CNN
+F 1 "+3.3V" H 4400 3560 30  0000 C CNN
+F 2 "" H 4400 3450 60  0000 C CNN
+F 3 "" H 4400 3450 60  0000 C CNN
+	1    4400 3450
+	1    0    0    -1
+$EndComp
+$Comp
+L GND #PWR?
+U 1 1 514F73D3
+P 4400 3850
+F 0 "#PWR?" H 4400 3850 30  0001 C CNN
+F 1 "GND" H 4400 3780 30  0001 C CNN
+F 2 "" H 4400 3850 60  0000 C CNN
+F 3 "" H 4400 3850 60  0000 C CNN
+	1    4400 3850
+	1    0    0    -1
+$EndComp
+$Comp
+L GND #PWR?
+U 1 1 514F73E2
+P 4400 4800
+F 0 "#PWR?" H 4400 4800 30  0001 C CNN
+F 1 "GND" H 4400 4730 30  0001 C CNN
+F 2 "" H 4400 4800 60  0000 C CNN
+F 3 "" H 4400 4800 60  0000 C CNN
+	1    4400 4800
+	1    0    0    -1
+$EndComp
 $EndSCHEMATC
